Commit message: added route, ground, profile

File: src/gnssd_description/urdf/robot.urdf.xacro (robot description, xacro)
@@ -13,4 +13,5 @@
     DiffDrive            /cmd_vel in, /odom_raw out (its TF is NOT used, see CLAUDE.md)
     JointStatePublisher  /joint_states, so robot_state_publisher can move the wheels
+    OdometryPublisher    /ground_truth, exact world pose for evaluation (TF not used)
   All numbers come from robot_params.xacro.
 -->
@@ -78,6 +79,13 @@
         <material name="wheel_black"/>
       </visual>
+      <!-- Collision is a SPHERE of the wheel radius, not the cylinder.
+           A cylinder lying on the floor touches it along an edge, and the
+           physics engine puts the contact near the inner rim: the effective
+           track width becomes ~0.23 m instead of 0.26 m, and the robot turns
+           ~10 % faster than DiffDrive assumes (measured in Step 2). A sphere
+           touches the floor in exactly one point in the wheel's mid-plane,
+           so the real kinematics match wheel_separation. -->
       <collision>
-        <geometry><cylinder radius="${wheel_radius}" length="${wheel_width}"/></geometry>
+        <geometry><sphere radius="${wheel_radius}"/></geometry>
       </collision>
       <xacro:cylinder_inertial mass="${wheel_mass}" radius="${wheel_radius}"
@@ -243,4 +251,18 @@
       <topic>joint_states</topic>
     </plugin>
+    <!-- Ground truth for evaluation (/ground_truth). In gz-sim 8 this system
+         publishes the model's WORLD pose (no initial pose is subtracted), so
+         the frame is called "world". No noise is added. Like DiffDrive, it
+         always publishes a TF message; that topic is not bridged. -->
+    <plugin filename="gz-sim-odometry-publisher-system"
+            name="gz::sim::systems::OdometryPublisher">
+      <odom_topic>ground_truth</odom_topic>
+      <odom_frame>world</odom_frame>
+      <robot_base_frame>base_link</robot_base_frame>
+      <odom_publish_frequency>${ground_truth_publish_rate}</odom_publish_frequency>
+      <dimensions>2</dimensions>
+      <gaussian_noise>0.0</gaussian_noise>
+      <tf_topic>gz_ground_truth_tf_not_bridged</tf_topic>
+    </plugin>
   </gazebo>
 </robot>

File: src/gnssd_description/urdf/robot_params.xacro (robot description, xacro)
@@ -63,3 +63,5 @@
   <!-- ===================== Drive controller ===================== -->
   <xacro:property name="odom_publish_rate" value="50"/>   <!-- Hz, /odom_raw -->
+  <!-- ===================== Ground truth ===================== -->
+  <xacro:property name="ground_truth_publish_rate" value="50"/>   <!-- Hz, /ground_truth -->
 </robot>

Commit message: imu model, ekf base

File: src/gnssd_description/urdf/robot.urdf.xacro (robot description, xacro)
@@ -191,6 +191,8 @@
     </sensor>
   </gazebo>
-  <!-- Noise block shared by the three gyro axes and by the three accelerometer axes. -->
-  <xacro:macro name="imu_axis_noise" params="axis stddev bias_mean bias_stddev">
+  <!-- Noise block shared by the three gyro axes and by the three accelerometer axes.
+       The dynamic (in-run) bias is optional; 0 switches it off. -->
+  <xacro:macro name="imu_axis_noise"
+               params="axis stddev bias_mean bias_stddev dynamic_bias_stddev:=0.0 dynamic_bias_corr_time:=0.0">
     <xacro:element xacro:name="${axis}">
       <noise type="gaussian">
@@ -199,4 +201,6 @@
         <bias_mean>${bias_mean}</bias_mean>
         <bias_stddev>${bias_stddev}</bias_stddev>
+        <dynamic_bias_stddev>${dynamic_bias_stddev}</dynamic_bias_stddev>
+        <dynamic_bias_correlation_time>${dynamic_bias_corr_time}</dynamic_bias_correlation_time>
       </noise>
     </xacro:element>
@@ -211,9 +215,15 @@
         <angular_velocity>
           <xacro:imu_axis_noise axis="x" stddev="${imu_gyro_noise_stddev}"
-              bias_mean="${imu_gyro_bias_mean}" bias_stddev="${imu_gyro_bias_stddev}"/>
+              bias_mean="${imu_gyro_bias_mean}" bias_stddev="${imu_gyro_bias_stddev}"
+              dynamic_bias_stddev="${imu_gyro_dynamic_bias_stddev}"
+              dynamic_bias_corr_time="${imu_gyro_dynamic_bias_corr_time}"/>
           <xacro:imu_axis_noise axis="y" stddev="${imu_gyro_noise_stddev}"
-              bias_mean="${imu_gyro_bias_mean}" bias_stddev="${imu_gyro_bias_stddev}"/>
+              bias_mean="${imu_gyro_bias_mean}" bias_stddev="${imu_gyro_bias_stddev}"
+              dynamic_bias_stddev="${imu_gyro_dynamic_bias_stddev}"
+              dynamic_bias_corr_time="${imu_gyro_dynamic_bias_corr_time}"/>
           <xacro:imu_axis_noise axis="z" stddev="${imu_gyro_noise_stddev}"
-              bias_mean="${imu_gyro_bias_mean}" bias_stddev="${imu_gyro_bias_stddev}"/>
+              bias_mean="${imu_gyro_bias_mean}" bias_stddev="${imu_gyro_bias_stddev}"
+              dynamic_bias_stddev="${imu_gyro_dynamic_bias_stddev}"
+              dynamic_bias_corr_time="${imu_gyro_dynamic_bias_corr_time}"/>
         </angular_velocity>
         <linear_acceleration>

File: src/gnssd_description/urdf/robot_params.xacro (robot description, xacro)
@@ -52,10 +52,28 @@
   <xacro:property name="imu_z_offset" value="0.02"/>
   <xacro:property name="imu_update_rate" value="100"/>   <!-- Hz -->
-  <!-- PLACEHOLDER noise values. They will be replaced with numbers taken
-       from the datasheet of the real IMU. In Gazebo the bias is drawn once
-       at start-up from N(bias_mean, bias_stddev) and then stays constant. -->
-  <xacro:property name="imu_gyro_noise_stddev"  value="0.005"/>    <!-- rad/s -->
-  <xacro:property name="imu_gyro_bias_mean"     value="0.0005"/>   <!-- rad/s -->
-  <xacro:property name="imu_gyro_bias_stddev"   value="0.0001"/>   <!-- rad/s -->
+  <!-- Gyroscope: model of a CALIBRATED MEMS gyro of the Bosch BMI088 class.
+       White noise. Datasheet noise density ~0.014 deg/s/sqrt(Hz). The IMU
+       publishes at 100 Hz, so the bandwidth is ~50 Hz:
+         0.014 deg/s/sqrt(Hz) * sqrt(50 Hz) = 0.099 deg/s = 0.0017 rad/s.
+       Bias. The large turn-on offset of a MEMS gyro is assumed to be removed
+       before every run by averaging the gyro while the robot stands still.
+       What remains is a small residual, modelled as
+         bias_mean = 0, bias_stddev = 1.0e-4 rad/s (about 0.02 deg/s).
+       Gazebo draws this bias once per run from N(bias_mean, bias_stddev)
+       (with a random sign) and keeps it; the seed option of gz sim makes the draw
+       repeatable, see sim.launch.py.
+       In-run bias instability (dynamic bias). BMI088 class: ~2 deg/h
+       = 1e-5 rad/s. gz-sensors 8 supports it as a first-order Gauss-Markov
+       process (dynamic_bias_stddev, dynamic_bias_correlation_time). The
+       correlation time is chosen longer than a run, so it acts as a slow
+       drift of the bias. -->
+  <xacro:property name="imu_gyro_noise_stddev"            value="0.0017"/>   <!-- rad/s -->
+  <xacro:property name="imu_gyro_bias_mean"               value="0.0"/>      <!-- rad/s -->
+  <xacro:property name="imu_gyro_bias_stddev"             value="1.0e-4"/>   <!-- rad/s -->
+  <xacro:property name="imu_gyro_dynamic_bias_stddev"     value="1.0e-5"/>   <!-- rad/s -->
+  <xacro:property name="imu_gyro_dynamic_bias_corr_time"  value="1000.0"/>   <!-- s -->
+  <!-- Accelerometer: NOT FUSED BY THE EKF (only the gyro z rate is used).
+       The values are the old placeholders and only matter if the
+       accelerometer is used later. -->
   <xacro:property name="imu_accel_noise_stddev" value="0.02"/>     <!-- m/s^2 -->
   <xacro:property name="imu_accel_bias_mean"    value="0.01"/>     <!-- m/s^2 -->

Commit message: fix gyro

File: src/gnssd_description/urdf/robot.urdf.xacro (robot description, xacro)
@@ -206,4 +206,8 @@
     </xacro:element>
   </xacro:macro>
+  <!-- gz-sensors parameter for the gyro drift: the stationary value from
+       robot_params.xacro divided by sqrt(tau / 2) (see the note there). -->
+  <xacro:property name="gyro_dynamic_bias_sigma_gz"
+                  value="${imu_gyro_dynamic_bias_stddev / (imu_gyro_dynamic_bias_corr_time / 2) ** 0.5}"/>
   <gazebo reference="imu_link">
     <sensor name="imu" type="imu">
@@ -216,13 +220,13 @@
           <xacro:imu_axis_noise axis="x" stddev="${imu_gyro_noise_stddev}"
               bias_mean="${imu_gyro_bias_mean}" bias_stddev="${imu_gyro_bias_stddev}"
-              dynamic_bias_stddev="${imu_gyro_dynamic_bias_stddev}"
+              dynamic_bias_stddev="${gyro_dynamic_bias_sigma_gz}"
               dynamic_bias_corr_time="${imu_gyro_dynamic_bias_corr_time}"/>
           <xacro:imu_axis_noise axis="y" stddev="${imu_gyro_noise_stddev}"
               bias_mean="${imu_gyro_bias_mean}" bias_stddev="${imu_gyro_bias_stddev}"
-              dynamic_bias_stddev="${imu_gyro_dynamic_bias_stddev}"
+              dynamic_bias_stddev="${gyro_dynamic_bias_sigma_gz}"
               dynamic_bias_corr_time="${imu_gyro_dynamic_bias_corr_time}"/>
           <xacro:imu_axis_noise axis="z" stddev="${imu_gyro_noise_stddev}"
               bias_mean="${imu_gyro_bias_mean}" bias_stddev="${imu_gyro_bias_stddev}"
-              dynamic_bias_stddev="${imu_gyro_dynamic_bias_stddev}"
+              dynamic_bias_stddev="${gyro_dynamic_bias_sigma_gz}"
               dynamic_bias_corr_time="${imu_gyro_dynamic_bias_corr_time}"/>
         </angular_velocity>

File: src/gnssd_description/urdf/robot_params.xacro (robot description, xacro)
@@ -67,9 +67,16 @@
        process (dynamic_bias_stddev, dynamic_bias_correlation_time). The
        correlation time is chosen longer than a run, so it acts as a slow
-       drift of the bias. -->
+       drift of the bias.
+       NOTE (fixed in Step 4): gz-sensors' dynamic_bias_stddev is NOT the
+       stationary standard deviation of the drift. Its update is
+         b(k+1) = exp(-dt/tau) b(k) + N(0, sigma_gz^2 tau/2 (1 - exp(-2 dt/tau))),
+       whose stationary standard deviation is sigma_gz * sqrt(tau / 2).
+       imu_gyro_dynamic_bias_stddev below is the physical (stationary) value;
+       robot.urdf.xacro converts it: sigma_gz = value / sqrt(tau / 2).
+       Step 3 passed 1e-5 directly, i.e. a stationary drift of 2.2e-4 rad/s. -->
   <xacro:property name="imu_gyro_noise_stddev"            value="0.0017"/>   <!-- rad/s -->
   <xacro:property name="imu_gyro_bias_mean"               value="0.0"/>      <!-- rad/s -->
   <xacro:property name="imu_gyro_bias_stddev"             value="1.0e-4"/>   <!-- rad/s -->
-  <xacro:property name="imu_gyro_dynamic_bias_stddev"     value="1.0e-5"/>   <!-- rad/s -->
+  <xacro:property name="imu_gyro_dynamic_bias_stddev"     value="1.0e-5"/>   <!-- rad/s, stationary -->
   <xacro:property name="imu_gyro_dynamic_bias_corr_time"  value="1000.0"/>   <!-- s -->
   <!-- Accelerometer: NOT FUSED BY THE EKF (only the gyro z rate is used).
